File: PCB/Spotwelderix-controlboard/_autosave-Spotwelderix-controlboard.sch (KiCad schematic (older format))
At the start: 35 parts, among them J1 ChargerPower, J2 LEDs, J3 ExtPwr_FAn, P1 Display, P2 CONN_01X08, Q1 AO3400A, Q2 AO3400A, Q5 AO3400A, U1 NodeMCU32, U3 LM7805M_TO263

Commit message: pcb update 1.9
Parts:
- added C? (x2): 10n, Capacitor_SMD:C_0805_2012Metric, symbol Spotwelderix-controlboard-rescue:C-Device
- added R? (x2): 10k, Resistor_SMD:R_0805_2012Metric, symbol Arduino_Spot_Welderparts:R
- BZ1: symbol Device:Buzzer -> Spotwelderix-controlboard-rescue:Buzzer-Device
- C1, C2, C3, C5, C6, C7: symbol Device:C -> Spotwelderix-controlboard-rescue:C-Device
- C4: symbol Device:CP -> Spotwelderix-controlboard-rescue:CP-Device
- H1, H2, H3, H4: symbol Mechanical:MountingHole -> Spotwelderix-controlboard-rescue:MountingHole-Mechanical
- J1: symbol Connector:Conn_01x05_Male -> Spotwelderix-controlboard-rescue:Conn_01x05_Male-Connector
- J2: symbol Connector:Conn_01x03_Male -> Spotwelderix-controlboard-rescue:Conn_01x03_Male-Connector
- P2: symbol Connector:Conn_01x09_Male -> Spotwelderix-controlboard-rescue:Conn_01x09_Male-Connector
- Q1, Q2, Q5: symbol Transistor_FET:AO3400A -> Spotwelderix-controlboard-rescue:AO3400A-Transistor_FET
- R11, R6, R8: value 33k -> 15k
- R12, R7, R9: value 10k -> 2.5k
- U3: symbol Regulator_Linear:LM7805_TO220 -> Spotwelderix-controlboard-rescue:LM7805_TO220-Regulator_Linear
Connections:
- net +3V3: now also R?.1, R?.1
- net BUZZ: now also R?.2
- net FAN: now also R?.2
- net GND: now also C?.2, C?.2
- net ProbeADC: now also C?.1
- net VCC_ADC: now also C?.1
Other:
- note added: "6.5 kHz"
- moved on the sheet: R11, R12, R8, R9
