File: PCB/Spotwelderix-controlboard/Spotwelderix-controlboard.sch (KiCad schematic (older format))
At the start: 27 parts, among them J1 Extender, J3 Switch_OnOFF, J4 FAN, P1 Display, P2 CONN_01X08, Q1 DMG1012T-7, Q2 DMG1012T-7, U1 NodeMCU32, U2 ADS1115_Module, U3 LM7805M_TO263

Commit message: power pcb added
Parts:
- added C6: 10n, Capacitor_SMD:C_0805_2012Metric, symbol Device:C
- added D2: D, Diode_SMD:D_1206_3216Metric, symbol Arduino_Spot_Welderparts:D
- added H1, H2, H3, H4: MountingHole, MountingHole:MountingHole_3.2mm_M3_DIN965_Pad_TopBottom, symbol Mechanical:MountingHole
Connections:
- net labels added: A2_ProbeADC, A3_VCC_ADC
- wire segments 121 -> 138
- no-connect marks 16 -> 14
Other:
- moved on the sheet: R3, R6
Changed lines of the file:
@@
 	5500 1650 5500 1750
 Wire Wire Line
-	5500 2050 5500 2150
+	5500 2050 5500 2100
 Wire Wire Line
 	6300 2150 5500 2150
@@
 	9200 3100 9500 3100
 $Comp
-L power:+5V #PWR0109
-U 1 1 604BBC57
-P 9800 2400
-F 0 "#PWR0109" H 9800 2250 50  0001 C CNN
-F 1 "+5V" H 9815 2573 50  0000 C CNN
-F 2 "" H 9800 2400 50  0001 C CNN
-F 3 "" H 9800 2400 50  0001 C CNN
-	1    9800 2400
-	1    0    0    -1
-$EndComp
-$Comp
 L Connector:Conn_01x02_Male J4
 U 1 1 604C477C
@@
 Wire Wire Line
 	3050 5550 3050 5800
+Text GLabel 4600 3550 2    50   Input ~ 0
+SCL
 Text GLabel 4600 3650 2    50   Input ~ 0
-SCL
-Text GLabel 4600 3550 2    50   Input ~ 0
 SDA
 Wire Wire Line
@@
 Wire Wire Line
 	4500 3650 4600 3650
-Text GLabel 1700 4700 0    50   Input ~ 0
+Text GLabel 1850 4900 0    50   Input ~ 0
 Dallas
-Text GLabel 1850 4900 0    50   Input ~ 0
+Text GLabel 1200 4700 0    50   Input ~ 0
 Gate_logic
-Wire Wire Line
-	1700 4700 2150 4700
 Wire Wire Line
 	2150 4900 1850 4900
@@
 F 1 "EC12D1524403 " H 2450 1800 60  0000 C CNN
 F 2 "Rotary_Encoder:RotaryEncoder_Alps_EC12E-Switch_Vertical_H20mm" H 2600 1400 60  0001 C CNN
-F 3 "https://www.mouser.de/ProductDetail/Alps-Alpine/EC12D1524403/?qs=%2Fha2pyFadujS61L3lQIIqGKdqySEQUGy9PSQHwezRaem1G6obKDSmg%3D%3D" H 2600 1400 60  0000 C CNN
+F 3 "https://www.mouser.de/ProductDetail/Alps-Alpine/EC12D1524403/?qs=%2Fha2pyFadujS61L3lQIIqGKdqySEQUGy9PSQHwezRaem1G6obKDSmg%3D%3D" H 2600 1400 60  0001 C CNN
 	1    2600 1400
 	1    0    0    -1
@@
 L Arduino_Spot_Welderparts:R R6
 U 1 1 601B227D
-P 5150 2000
-F 0 "R6" H 5220 2046 50  0000 L CNN
-F 1 "33k" H 5220 1955 50  0000 L CNN
-F 2 "Resistor_SMD:R_0805_2012Metric" V 5080 2000 50  0001 C CNN
-F 3 "" H 5150 2000 50  0000 C CNN
-	1    5150 2000
+P 5150 1900
+F 0 "R6" H 5220 1946 50  0000 L CNN
+F 1 "33k" H 5220 1855 50  0000 L CNN
+F 2 "Resistor_SMD:R_0805_2012Metric" V 5080 1900 50  0001 C CNN
+F 3 "" H 5150 1900 50  0000 C CNN
+	1    5150 1900
 	1    0    0    -1
 $EndComp
@@
 	5100 1650 5150 1650
 Wire Wire Line
-	5150 1650 5150 1850
-Wire Wire Line
-	5150 2150 5150 2250
+	5150 1650 5150 1750
+Wire Wire Line
+	5150 2050 5150 2200
 Wire Wire Line
 	5500 2150 5500 2300
@@
 Text GLabel 3900 1150 2    50   Input ~ 0
 UI_RotEnc_A
-Text GLabel 3850 1650 2    50   Input ~ 0
+Text GLabel 4000 1650 2    50   Input ~ 0
 UI_RotEnc_B
 $Comp
 L Arduino_Spot_Welderparts:R R3
 U 1 1 601DF3B0
-P 3550 1650
-F 0 "R3" H 3620 1696 50  0000 L CNN
-F 1 "100" H 3620 1605 50  0000 L CNN
-F 2 "Resistor_SMD:R_0805_2012Metric" H 3620 1559 50  0001 L CNN
-F 3 "" H 3550 1650 50  0001 C CNN
-	1    3550 1650
+P 3700 1650
+F 0 "R3" H 3770 1696 50  0000 L CNN
+F 1 "100" H 3770 1605 50  0000 L CNN
+F 2 "Resistor_SMD:R_0805_2012Metric" H 3770 1559 50  0001 L CNN
+F 3 "" H 3700 1650 50  0001 C CNN
+	1    3700 1650
 	0    1    1    0
 $EndComp
@@
 Wire Wire Line
 	3150 1650 3250 1650
-Wire Wire Line
-	3400 1650 3250 1650
 Connection ~ 3250 1650
 Wire Wire Line
@@
 	3250 800  3700 800
 Wire Wire Line
-	3700 1650 3850 1650
+	3850 1650 4000 1650
 $Comp
 L Arduino_Spot_Welderparts:R R1
@@
 NoConn ~ 6300 1850
 NoConn ~ 2150 3500
-NoConn ~ 2150 3600
-NoConn ~ 2150 3700
 NoConn ~ 4100 3750
 NoConn ~ 4100 3850
@@
 	8850 1100 8850 1250
 Wire Wire Line
-	8550 1250 8750 1250
+	8550 1250 8600 1250
 Connection ~ 8850 1250
 Wire Wire Line
@@
 Wire Wire Line
 	9850 1600 9850 1750
+$Comp
+L Mechanical:MountingHole H1
+U 1 1 60212773
+P 7200 6350
+F 0 "H1" H 7300 6396 50  0000 L CNN
+F 1 "MountingHole" H 7300 6305 50  0000 L CNN
+F 2 "MountingHole:MountingHole_3.2mm_M3_DIN965_Pad_TopBottom" H 7200 6350 50  0001 C CNN
+F 3 "~" H 7200 6350 50  0001 C CNN
+	1    7200 6350
+	1    0    0    -1
+$EndComp
+$Comp
+L Mechanical:MountingHole H2
+U 1 1 602345BB
+P 8050 6350
+F 0 "H2" H 8150 6396 50  0000 L CNN
+F 1 "MountingHole" H 8150 6305 50  0000 L CNN
+F 2 "MountingHole:MountingHole_3.2mm_M3_DIN965_Pad_TopBottom" H 8050 6350 50  0001 C CNN
+F 3 "~" H 8050 6350 50  0001 C CNN
+	1    8050 6350
+	1    0    0    -1
+$EndComp
+$Comp
+L Mechanical:MountingHole H3
+U 1 1 60238BE0
+P 8900 6350
+F 0 "H3" H 9000 6396 50  0000 L CNN
+F 1 "MountingHole" H 9000 6305 50  0000 L CNN
+F 2 "MountingHole:MountingHole_3.2mm_M3_DIN965_Pad_TopBottom" H 8900 6350 50  0001 C CNN
+F 3 "~" H 8900 6350 50  0001 C CNN
+	1    8900 6350
+	1    0    0    -1
+$EndComp
+$Comp
+L Mechanical:MountingHole H4
+U 1 1 6023D34D
+P 9750 6350
+F 0 "H4" H 9850 6396 50  0000 L CNN
+F 1 "MountingHole" H 9850 6305 50  0000 L CNN
+F 2 "MountingHole:MountingHole_3.2mm_M3_DIN965_Pad_TopBottom" H 9750 6350 50  0001 C CNN
+F 3 "~" H 9750 6350 50  0001 C CNN
+	1    9750 6350
+	1    0    0    -1
+$EndComp
+Wire Wire Line
+	9800 2400 9250 2400
+Wire Wire Line
+	8600 2400 8600 1250
+Connection ~ 8600 1250
+Wire Wire Line
+	8600 1250 8750 1250
+$Comp
+L Arduino_Spot_Welderparts:D D2
+U 1 1 60173424
+P 9250 2600
+F 0 "D2" H 9250 2385 50  0000 C CNN
+F 1 "D" H 9250 2476 50  0000 C CNN
+F 2 "Diode_SMD:D_1206_3216Metric" H 9250 2600 50  0001 C CNN
+F 3 "" H 9250 2600 50  0000 C CNN
+	1    9250 2600
+	0    1    1    0
+$EndComp
+Wire Wire Line
+	9250 2750 9550 2750
+Wire Wire Line
+	9550 2750 9550 2650
+Wire Wire Line
+	9550 2650 9800 2650
+Connection ~ 9800 2650
+Wire Wire Line
+	9250 2450 9250 2400
+Connection ~ 9250 2400
+Wire Wire Line
+	9250 2400 8600 2400
+Wire Wire Line
+	1200 4700 1400 4700
+$Comp
+L Device:C C6
+U 1 1 6018E2B1
+P 1400 5050
+F 0 "C6" H 1515 5096 50  0000 L CNN
+F 1 "10n" H 1515 5005 50  0000 L CNN
+F 2 "Capacitor_SMD:C_0805_2012Metric" H 1438 4900 50  0001 C CNN
+F 3 "https://www.mouser.de/ProductDetail/Samsung-Electro-Mechanics/CL31A106KBHNNNE/?qs=sGAEpiMZZMuMW9TJLBQkXpvci%252BYHLlg21rnqFxf28Ww%3D" H 1400 5050 50  0001 C CNN
+	1    1400 5050
+	1    0    0    -1
+$EndComp
+$Comp
+L power:GND #PWR01
+U 1 1 6019341A
+P 1400 5300
+F 0 "#PWR01" H 1400 5050 50  0001 C CNN
+F 1 "GND" H 1405 5127 50  0000 C CNN
+F 2 "" H 1400 5300 50  0001 C CNN
+F 3 "" H 1400 5300 50  0001 C CNN
+	1    1400 5300
+	1    0    0    -1
+$EndComp
+Wire Wire Line
+	1400 4700 1400 4900
+Connection ~ 1400 4700
+Wire Wire Line
+	1400 4700 2150 4700
+Wire Wire Line
+	1400 5200 1400 5300
+Wire Wire Line
+	3250 1650 3550 1650
+Text GLabel 4850 2100 0    50   Input ~ 0
+A2_ProbeADC
+Text GLabel 4850 2200 0    50   Input ~ 0
+A3_VCC_ADC
+Wire Wire Line
+	4850 2100 5500 2100
+Connection ~ 5500 2100
+Wire Wire Line
+	5500 2100 5500 2150
+Wire Wire Line
+	4850 2200 5150 2200
+Connection ~ 5150 2200
+Wire Wire Line
+	5150 2200 5150 2250
+Text GLabel 1750 3600 0    50   Input ~ 0
+A2_ProbeADC
+Text GLabel 1750 3700 0    50   Input ~ 0
+A3_VCC_ADC
+Wire Wire Line
+	1750 3600 2150 3600
+Wire Wire Line
+	1750 3700 2150 3700
 $EndSCHEMATC

Commit message: power pcb updated, added safe power for driver
Parts:
- D1, D2: footprint Diode_SMD:D_1206_3216Metric -> Diode_SMD:D_SMA
- J1: footprint Connector_JST:JST_XH_B6B-XH-A_1x06_P2.50mm_Vertical -> Connector_JST:JST_XH_S6B-XH-A-1_1x06_P2.50mm_Horizontal
Changed lines of the file:
@@
 F 0 "D1" H 8400 1035 50  0000 C CNN
 F 1 "D" H 8400 1126 50  0000 C CNN
-F 2 "Diode_SMD:D_1206_3216Metric" H 8400 1250 50  0001 C CNN
+F 2 "Diode_SMD:D_SMA" H 8400 1250 50  0001 C CNN
 F 3 "" H 8400 1250 50  0000 C CNN
 	1    8400 1250
@@
 F 0 "J1" H 4672 5624 50  0000 R CNN
 F 1 "Extender" H 4672 5533 50  0000 R CNN
-F 2 "Connector_JST:JST_XH_B6B-XH-A_1x06_P2.50mm_Vertical" H 4700 5650 50  0001 C CNN
+F 2 "Connector_JST:JST_XH_S6B-XH-A-1_1x06_P2.50mm_Horizontal" H 4700 5650 50  0001 C CNN
 F 3 "~" H 4700 5650 50  0001 C CNN
 	1    4700 5650
@@
 F 0 "D2" H 9250 2385 50  0000 C CNN
 F 1 "D" H 9250 2476 50  0000 C CNN
-F 2 "Diode_SMD:D_1206_3216Metric" H 9250 2600 50  0001 C CNN
+F 2 "Diode_SMD:D_SMA" H 9250 2600 50  0001 C CNN
 F 3 "" H 9250 2600 50  0000 C CNN
 	1    9250 2600

Commit message: ena powerpcb added
Parts:
- removed J1: Extender, Connector_JST:JST_XH_S6B-XH-A-1_1x06_P2.50mm_Horizontal, symbol Connector:Conn_01x06_Male
- added C7: 100n, Capacitor_SMD:C_0805_2012Metric, symbol Device:C
- added D3: D, Diode_SMD:D_SMA, symbol Arduino_Spot_Welderparts:D
- added D4: 3.6V, Diode_SMD:D_SOD-323_HandSoldering, symbol Device:D_Zener
- added J2: LEDs, Connector_JST:JST_XH_B3B-XH-A_1x03_P2.50mm_Vertical, symbol Connector:Conn_01x03_Male
- added Q3, Q4: DMG1012T-7, SamacSys_Parts:SOT50P160X80-3N, symbol SamacSys_Parts:DMG1012T-7
- added R10, R12: 10k, Resistor_SMD:R_0805_2012Metric, symbol Arduino_Spot_Welderparts:R
- added R11, R13: 100, Resistor_SMD:R_0805_2012Metric, symbol Arduino_Spot_Welderparts:R
- C1, C2, C3: value 100n -> 100p
- J3: footprint Connector_JST:JST_XH_B2B-XH-A_1x02_P2.50mm_Vertical -> Connector_JST:JST_XH_B7B-XH-A_1x07_P2.50mm_Vertical; symbol Connector:Conn_01x02_Male -> Connector:Conn_01x07_Male
- J4: value FAN -> Int_Charger_supply
Connections:
- net labels added: ChargDisEna, ExtPower, Ext_Trigger, FAN_GND, LED, LM7805_in
- net labels removed: PowerVCC
- wire segments 138 -> 170
- no-connect marks 14 -> 15
Other:
- note added: "ExtConn: Ext+m, Ext-, Powerswitch1,2, Fan+, Fan-, ExtTrig\n"
- moved on the sheet: BZ1, C1, C2, C3, C4, C5, D1, D2, P2, U3

Commit message: ordered version v01
Parts:
- removed D1: D, Diode_SMD:D_SMA, symbol Arduino_Spot_Welderparts:D
- removed D4: 3.6V, Diode_SMD:D_SOD-323_HandSoldering, symbol Device:D_Zener
- removed J4: Int_Charger_supply, Connector_JST:JST_XH_B2B-XH-A_1x02_P2.50mm_Vertical, symbol Connector:Conn_01x02_Male
- removed Q1, Q2, Q3, Q4: DMG1012T-7, SamacSys_Parts:SOT50P160X80-3N, symbol SamacSys_Parts:DMG1012T-7
- removed R10: 10k, Resistor_SMD:R_0805_2012Metric, symbol Arduino_Spot_Welderparts:R
- removed R13: 100, Resistor_SMD:R_0805_2012Metric, symbol Arduino_Spot_Welderparts:R
- removed R4, R5: 3k3, Resistor_SMD:R_0805_2012Metric, symbol Arduino_Spot_Welderparts:R
- removed U2: ADS1115_Module, Connector_PinHeader_2.54mm:PinHeader_1x10_P2.54mm_Vertical, symbol my_parts:ADS1115_Module
- added J1: ChargerPower, Connector_JST:JST_XH_S5B-XH-A_1x05_P2.50mm_Horizontal, symbol Connector:Conn_01x05_Male
- added Q1, Q2, Q5: AO3400A, Package_TO_SOT_SMD:SOT-23, symbol Transistor_FET:AO3400A
- added R14: 100, Resistor_SMD:R_0805_2012Metric, symbol Arduino_Spot_Welderparts:R
- C7: value 100n -> 100p
- J3: value Switch_OnOFF -> ExtPwr_FAn; footprint Connector_JST:JST_XH_B7B-XH-A_1x07_P2.50mm_Vertical -> Connector_JST:JST_XH_B4B-XH-A_1x04_P2.50mm_Vertical; symbol Connector:Conn_01x07_Male -> Arduino_Spot_Welderparts:CONN_01X04
- P1: footprint Connector_JST:JST_XH_B8B-XH-A_1x08_P2.50mm_Vertical -> Connector_JST:JST_XH_S8B-XH-A_1x08_P2.50mm_Horizontal
- P2: footprint Connector_JST:JST_XH_B8B-XH-A_1x08_P2.50mm_Vertical -> Connector_JST:JST_XH_B9B-XH-A_1x09_P2.50mm_Vertical; symbol Arduino_Spot_Welderparts:CONN_01X08 -> Connector:Conn_01x09_Male
- R11: value 100 -> 33k
Connections:
- net labels added: ChargerEna, EnableSupply, ExtPWRADC, FootSwitch, ProbeADC, Shuntvoltage, VCC_ADC, Vbat_ADC
- net labels removed: A2_ProbeADC, A3_VCC_ADC, ChargDisEna, Ext_Trigger, R_Schunt_H, R_Schunt_L, SCL, SDA
- wire segments 170 -> 141
- no-connect marks 15 -> 12
Other:
- note added: "ExtConn: Ext+, Ext-,Fan+, Fan-,\n"
- note removed: "ExtConn: Ext+m, Ext-, Powerswitch1,2, Fan+, Fan-, ExtTrig\n"
- moved on the sheet: C4, C5, D2, D3, R6, R8, R9, U3

Commit message: pcb update 1.9
Parts:
- added C? (x2): 10n, Capacitor_SMD:C_0805_2012Metric, symbol Device:C
- added R? (x2): 10k, Resistor_SMD:R_0805_2012Metric, symbol Arduino_Spot_Welderparts:R
- R11, R6, R8: value 33k -> 15k
- R12, R7, R9: value 10k -> 2.5k
- U1: symbol my_parts:NodeMCU32 -> Spotwelderix-controlboard-rescue:NodeMCU32-my_parts
Connections:
- net +3V3: now also R?.1, R?.1
- net BUZZ: now also R?.2
- net FAN: now also R?.2
- net GND: now also C?.2, C?.2
- net ProbeADC: now also C?.1
- net VCC_ADC: now also C?.1
Other:
- note added: "6.5 kHz"
- moved on the sheet: R11, R12, R8, R9
Changed lines of the file:
@@
 L Arduino_Spot_Welderparts:R R8
 U 1 1 603BCFB2
-P 5500 1700
-F 0 "R8" H 5570 1746 50  0000 L CNN
-F 1 "33k" H 5570 1655 50  0000 L CNN
-F 2 "Resistor_SMD:R_0805_2012Metric" V 5430 1700 50  0001 C CNN
-F 3 "" H 5500 1700 50  0000 C CNN
-	1    5500 1700
+P 5850 1700
+F 0 "R8" H 5920 1746 50  0000 L CNN
+F 1 "15k" H 5920 1655 50  0000 L CNN
+F 2 "Resistor_SMD:R_0805_2012Metric" V 5780 1700 50  0001 C CNN
+F 3 "" H 5850 1700 50  0000 C CNN
+	1    5850 1700
 	1    0    0    -1
 $EndComp
@@
 L Arduino_Spot_Welderparts:R R9
 U 1 1 603BE2C9
-P 5500 2500
-F 0 "R9" H 5570 2546 50  0000 L CNN
-F 1 "10k" H 5570 2455 50  0000 L CNN
-F 2 "Resistor_SMD:R_0805_2012Metric" H 5570 2409 50  0001 L CNN
-F 3 "" H 5500 2500 50  0001 C CNN
-	1    5500 2500
+P 5850 2500
+F 0 "R9" H 5920 2546 50  0000 L CNN
+F 1 "2.5k" H 5920 2455 50  0000 L CNN
+F 2 "Resistor_SMD:R_0805_2012Metric" H 5920 2409 50  0001 L CNN
+F 3 "" H 5850 2500 50  0001 C CNN
+	1    5850 2500
 	1    0    0    -1
 $EndComp
@@
 L power:VCC #PWR0107
 U 1 1 60423BF7
-P 5500 1450
-F 0 "#PWR0107" H 5500 1300 50  0001 C CNN
-F 1 "VCC" H 5515 1623 50  0000 C CNN
-F 2 "" H 5500 1450 50  0001 C CNN
-F 3 "" H 5500 1450 50  0001 C CNN
-	1    5500 1450
-	1    0    0    -1
-$EndComp
-Wire Wire Line
-	5500 1450 5500 1550
+P 5850 1450
+F 0 "#PWR0107" H 5850 1300 50  0001 C CNN
+F 1 "VCC" H 5865 1623 50  0000 C CNN
+F 2 "" H 5850 1450 50  0001 C CNN
+F 3 "" H 5850 1450 50  0001 C CNN
+	1    5850 1450
+	1    0    0    -1
+$EndComp
+Wire Wire Line
+	5850 1450 5850 1550
 $Comp
 L power:GND #PWR0108
 U 1 1 60458421
-P 5500 2700
-F 0 "#PWR0108" H 5500 2450 50  0001 C CNN
-F 1 "GND" H 5505 2527 50  0000 C CNN
-F 2 "" H 5500 2700 50  0001 C CNN
-F 3 "" H 5500 2700 50  0001 C CNN
-	1    5500 2700
-	1    0    0    -1
-$EndComp
-Wire Wire Line
-	5500 2700 5500 2650
+P 5850 2700
+F 0 "#PWR0108" H 5850 2450 50  0001 C CNN
+F 1 "GND" H 5855 2527 50  0000 C CNN
+F 2 "" H 5850 2700 50  0001 C CNN
+F 3 "" H 5850 2700 50  0001 C CNN
+	1    5850 2700
+	1    0    0    -1
+$EndComp
+Wire Wire Line
+	5850 2700 5850 2650
 Text GLabel 9550 3600 0    50   Input ~ 0
 FAN
 Wire Wire Line
-	9550 3600 9850 3600
+	9550 3600 9700 3600
 $Comp
 L power:GND #PWR0110
@@
 P 5150 1700
 F 0 "R6" H 5220 1746 50  0000 L CNN
-F 1 "33k" H 5220 1655 50  0000 L CNN
+F 1 "15k" H 5220 1655 50  0000 L CNN
 F 2 "Resistor_SMD:R_0805_2012Metric" V 5080 1700 50  0001 C CNN
 F 3 "" H 5150 1700 50  0000 C CNN
@@
 P 5150 2450
 F 0 "R7" H 5220 2496 50  0000 L CNN
-F 1 "10k" H 5220 2405 50  0000 L CNN
+F 1 "2.5k" H 5220 2405 50  0000 L CNN
 F 2 "Resistor_SMD:R_0805_2012Metric" H 5220 2359 50  0001 L CNN
 F 3 "" H 5150 2450 50  0001 C CNN
@@
 L power:GND #PWR0118
 U 1 1 601B2294
-P 5150 2700
-F 0 "#PWR0118" H 5150 2450 50  0001 C CNN
-F 1 "GND" H 5155 2527 50  0000 C CNN
-F 2 "" H 5150 2700 50  0001 C CNN
-F 3 "" H 5150 2700 50  0001 C CNN
-	1    5150 2700
-	1    0    0    -1
-$EndComp
-Wire Wire Line
-	5150 2700 5150 2600
+P 5150 2850
+F 0 "#PWR0118" H 5150 2600 50  0001 C CNN
+F 1 "GND" H 5155 2677 50  0000 C CNN
+F 2 "" H 5150 2850 50  0001 C CNN
+F 3 "" H 5150 2850 50  0001 C CNN
+	1    5150 2850
+	1    0    0    -1
+$EndComp
+Wire Wire Line
+	5150 2850 5150 2700
 Text GLabel 5100 1450 0    50   Input ~ 0
 Probe
@@
 BUZZ
 Wire Wire Line
-	4250 7100 4550 7100
+	4250 7100 4400 7100
 $Comp
 L power:+5V #PWR0132
@@
 Wire Wire Line
 	1400 5200 1400 5300
-Text GLabel 4850 2200 0    50   Input ~ 0
+Text GLabel 4800 2200 0    50   Input ~ 0
 ProbeADC
 Text GLabel 4850 2100 0    50   Input ~ 0
 VCC_ADC
-Wire Wire Line
-	4850 2100 5500 2100
-Connection ~ 5500 2100
-Wire Wire Line
-	4850 2200 5150 2200
+Connection ~ 5850 2100
+Wire Wire Line
+	4800 2200 4900 2200
 Connection ~ 5150 2200
 Wire Wire Line
@@
 	1400 1550 1500 1550
 Wire Wire Line
-	5500 2100 5500 2350
+	5850 2100 5850 2350
 Wire Wire Line
 	5150 2200 5150 2300
 $Comp
-L my_parts:NodeMCU32 U1
+L Spotwelderix-controlboard-rescue:NodeMCU32-my_parts U1
 U 1 1 601881C3
 P 3200 4250
@@
 	9750 4950 10200 4950
 Wire Wire Line
-	5500 1850 5500 2100
-Text GLabel 5850 1000 0    50   Input ~ 0
+	5850 1850 5850 2100
+Text GLabel 6250 1000 0    50   Input ~ 0
 ExtPower
-Wire Wire Line
-	4950 1950 5900 1950
 Text GLabel 4950 1950 0    50   Input ~ 0
 ExtPWRADC
 Wire Wire Line
-	5900 1950 5900 2400
-Connection ~ 5900 1950
-Wire Wire Line
-	5900 1000 5900 1550
-Wire Wire Line
-	5850 1000 5900 1000
-Wire Wire Line
-	5900 1850 5900 1950
-Wire Wire Line
-	5900 2750 5900 2700
+	6300 1950 6300 2400
+Connection ~ 6300 1950
+Wire Wire Line
+	6300 1000 6300 1550
+Wire Wire Line
+	6250 1000 6300 1000
+Wire Wire Line
+	6300 1850 6300 1950
+Wire Wire Line
+	6300 2750 6300 2700
 $Comp
 L power:GND #PWR010
 U 1 1 60319258
-P 5900 2750
-F 0 "#PWR010" H 5900 2500 50  0001 C CNN
-F 1 "GND" H 5905 2577 50  0000 C CNN
-F 2 "" H 5900 2750 50  0001 C CNN
-F 3 "" H 5900 2750 50  0001 C CNN
-	1    5900 2750
+P 6300 2750
+F 0 "#PWR010" H 6300 2500 50  0001 C CNN
+F 1 "GND" H 6305 2577 50  0000 C CNN
+F 2 "" H 6300 2750 50  0001 C CNN
+F 3 "" H 6300 2750 50  0001 C CNN
+	1    6300 2750
 	1    0    0    -1
 $EndComp
@@
 L Arduino_Spot_Welderparts:R R12
 U 1 1 6031924B
-P 5900 2550
-F 0 "R12" H 5970 2596 50  0000 L CNN
-F 1 "10k" H 5970 2505 50  0000 L CNN
-F 2 "Resistor_SMD:R_0805_2012Metric" H 5970 2459 50  0001 L CNN
-F 3 "" H 5900 2550 50  0001 C CNN
-	1    5900 2550
+P 6300 2550
+F 0 "R12" H 6370 2596 50  0000 L CNN
+F 1 "2.5k" H 6370 2505 50  0000 L CNN
+F 2 "Resistor_SMD:R_0805_2012Metric" H 6370 2459 50  0001 L CNN
+F 3 "" H 6300 2550 50  0001 C CNN
+	1    6300 2550
 	1    0    0    -1
 $EndComp
@@
 L Arduino_Spot_Welderparts:R R11
 U 1 1 60319245
-P 5900 1700
-F 0 "R11" H 5970 1746 50  0000 L CNN
-F 1 "33k" H 5970 1655 50  0000 L CNN
-F 2 "Resistor_SMD:R_0805_2012Metric" V 5830 1700 50  0001 C CNN
-F 3 "" H 5900 1700 50  0000 C CNN
-	1    5900 1700
+P 6300 1700
+F 0 "R11" H 6370 1746 50  0000 L CNN
+F 1 "15k" H 6370 1655 50  0000 L CNN
+F 2 "Resistor_SMD:R_0805_2012Metric" V 6230 1700 50  0001 C CNN
+F 3 "" H 6300 1700 50  0000 C CNN
+	1    6300 1700
 	1    0    0    -1
 $EndComp
@@
 Wire Wire Line
 	4850 6650 4850 6900
+$Comp
+L Arduino_Spot_Welderparts:R R?
+U 1 1 610D316C
+P 4400 6950
+F 0 "R?" H 4470 6996 50  0000 L CNN
+F 1 "10k" H 4470 6905 50  0000 L CNN
+F 2 "Resistor_SMD:R_0805_2012Metric" H 4470 6859 50  0001 L CNN
+F 3 "" H 4400 6950 50  0001 C CNN
+	1    4400 6950
+	1    0    0    -1
+$EndComp
+Connection ~ 4400 7100
+Wire Wire Line
+	4400 7100 4550 7100
+$Comp
+L Device:C C?
+U 1 1 610D9E59
+P 4900 2450
+F 0 "C?" H 4700 2500 50  0000 L CNN
+F 1 "10n" H 4650 2350 50  0000 L CNN
+F 2 "Capacitor_SMD:C_0805_2012Metric" H 4938 2300 50  0001 C CNN
+F 3 "https://www.mouser.de/ProductDetail/Samsung-Electro-Mechanics/CL31A106KBHNNNE/?qs=sGAEpiMZZMuMW9TJLBQkXpvci%252BYHLlg21rnqFxf28Ww%3D" H 4900 2450 50  0001 C CNN
+	1    4900 2450
+	1    0    0    -1
+$EndComp
+Wire Wire Line
+	4900 2300 4900 2200
+Connection ~ 4900 2200
+Wire Wire Line
+	4900 2200 5150 2200
+Wire Wire Line
+	4900 2600 4900 2700
+Wire Wire Line
+	4900 2700 5150 2700
+Connection ~ 5150 2700
+Wire Wire Line
+	5150 2700 5150 2600
+Wire Wire Line
+	4950 1950 6300 1950
+Wire Wire Line
+	4850 2100 5600 2100
+$Comp
+L Device:C C?
+U 1 1 61115154
+P 5600 2450
+F 0 "C?" H 5400 2500 50  0000 L CNN
+F 1 "10n" H 5350 2350 50  0000 L CNN
+F 2 "Capacitor_SMD:C_0805_2012Metric" H 5638 2300 50  0001 C CNN
+F 3 "https://www.mouser.de/ProductDetail/Samsung-Electro-Mechanics/CL31A106KBHNNNE/?qs=sGAEpiMZZMuMW9TJLBQkXpvci%252BYHLlg21rnqFxf28Ww%3D" H 5600 2450 50  0001 C CNN
+	1    5600 2450
+	1    0    0    -1
+$EndComp
+Wire Wire Line
+	5600 2300 5600 2100
+Connection ~ 5600 2100
+Wire Wire Line
+	5600 2100 5850 2100
+Wire Wire Line
+	5600 2600 5600 2700
+Wire Wire Line
+	5600 2700 5850 2700
+Connection ~ 5850 2700
+Text Notes 5400 2900 0    50   ~ 0
+6.5 kHz
+$Comp
+L power:+3V3 #PWR?
+U 1 1 61125D3E
+P 4400 6600
+F 0 "#PWR?" H 4400 6450 50  0001 C CNN
+F 1 "+3V3" H 4415 6773 50  0000 C CNN
+F 2 "" H 4400 6600 50  0001 C CNN
+F 3 "" H 4400 6600 50  0001 C CNN
+	1    4400 6600
+	1    0    0    -1
+$EndComp
+$Comp
+L power:+3V3 #PWR?
+U 1 1 6112C73B
+P 9700 3050
+F 0 "#PWR?" H 9700 2900 50  0001 C CNN
+F 1 "+3V3" H 9715 3223 50  0000 C CNN
+F 2 "" H 9700 3050 50  0001 C CNN
+F 3 "" H 9700 3050 50  0001 C CNN
+	1    9700 3050
+	1    0    0    -1
+$EndComp
+Wire Wire Line
+	9700 3050 9700 3200
+Wire Wire Line
+	4400 6600 4400 6800
+$Comp
+L Arduino_Spot_Welderparts:R R?
+U 1 1 61146B55
+P 9700 3350
+F 0 "R?" H 9770 3396 50  0000 L CNN
+F 1 "10k" H 9770 3305 50  0000 L CNN
+F 2 "Resistor_SMD:R_0805_2012Metric" H 9770 3259 50  0001 L CNN
+F 3 "" H 9700 3350 50  0001 C CNN
+	1    9700 3350
+	1    0    0    -1
+$EndComp
+Wire Wire Line
+	9700 3500 9700 3600
+Connection ~ 9700 3600
+Wire Wire Line
+	9700 3600 9850 3600
 $EndSCHEMATC
