File: PCB/Spotwelderix/Spotwelderix.sch (KiCad schematic (older format))
At the start: 41 parts

Commit message: power pcb added
Parts:
- removed C?: 470µ, symbol Device:CP
- removed C?: 10µ, Capacitor_SMD:C_1206_3216Metric, symbol Device:C
- removed C?: 100n, Capacitor_SMD:C_0805_2012Metric, symbol Device:C
- removed D?: D, symbol Arduino_Spot_Welderparts:D
- removed D? (x2): RF2001NS2D, Package_TO_SOT_SMD:TO-263-2_TabPin1, symbol Diode:C3D10060G
- removed J?: probe+, symbol Connector_Generic:Conn_01x01
- removed J? (x2): XT60, Connector_AMASS:AMASS_XT60-F_1x02_P7.20mm_Vertical, symbol Connector:Conn_01x02_Male
- removed J?: FAN, symbol Connector:Conn_01x02_Male
- removed Q?: DMG1012T-7, SOT50P160X80-3N, symbol SamacSys_Parts:DMG1012T-7
- removed R?: 33k, Resistor_SMD:R_0805_2012Metric, symbol Arduino_Spot_Welderparts:R
- removed R?: 10k, Resistor_SMD:R_0805_2012Metric, symbol Arduino_Spot_Welderparts:R
- removed U?: LM7805M_TO263, Package_TO_SOT_SMD:TO-263-3_TabPin2, symbol Regulator_Linear:LM7805_TO220
- removed U?: ADS1115_Module, symbol my_parts:ADS1115_Module
- added C11, C12, C13: 10µ, Capacitor_SMD:C_1206_3216Metric, symbol Device:C
- added H1, H3, H4, H5, H6: MountingHole_Pad, MountingHole:MountingHole_5.3mm_M5_Pad_Via, symbol Mechanical:MountingHole_Pad
- added H2, H7: MountingHole_Pad, MountingHole:MountingHole_3.2mm_M3_Pad_Via, symbol Mechanical:MountingHole_Pad
- added IC2, IC3: IXDD604SIA, SamacSys_Parts:SOIC127P600X175-8N, symbol SamacSys_Parts:IXDD604SIA
- added R2, R3, R4: 10k, Resistor_SMD:R_0805_2012Metric, symbol Arduino_Spot_Welderparts:R
- F1: renamed from F?; footprint (none) -> my_parts:ANL_Fuse
- IC1: renamed from IC?; footprint SOIC127P600X175-8N -> SamacSys_Parts:SOIC127P600X175-8N
- J4: renamed from J?; footprint (none) -> MountingHole:MountingHole_5.3mm_M5_Pad_Via
- P1: renamed from P?; footprint (none) -> Connector_JST:JST_XH_B8B-XH-A_1x08_P2.50mm_Vertical
- Q1, Q2, Q3, Q4, Q5, Q6, Q7, Q8: renamed from Q?; footprint Package_TO_SOT_THT:TO-220-3_Vertical -> Package_TO_SOT_SMD:TO-263-2
- gave numbers to parts that had none: 12
Connections:
- net labels added: FET_GND, Probe-
- net labels removed: FAN, SCL, SDA
- wire segments 183 -> 195
- no-connect marks 0 -> 6
Other:
- moved on the sheet: C1, C10, C2, C3, C4, C5, C6, C7, C8, C9, D1, D3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

Commit message: power pcb updated, added safe power for driver
Parts:
- added C14: 470µ, Capacitor_THT:CP_Radial_D10.0mm_P5.00mm, symbol Arduino_Spot_Welderparts:CP
- added D2: D, Diode_SMD:D_SMA, symbol Arduino_Spot_Welderparts:D
Connections:
- net labels added: VCCQ
- wire segments 195 -> 214
- no-connect marks 6 -> 0

Commit message: ena powerpcb added
Parts:
- removed C11: 10µ, Capacitor_SMD:C_1206_3216Metric, symbol Device:C
- removed IC1: IXDD604SIA, SamacSys_Parts:SOIC127P600X175-8N, symbol SamacSys_Parts:IXDD604SIA
- removed R2: 10k, Resistor_SMD:R_0805_2012Metric, symbol Arduino_Spot_Welderparts:R
- added J1: OnOffTast, Connector_JST:JST_XH_B2B-XH-A_1x02_P2.50mm_Vertical, symbol Connector:Conn_01x02_Male
- added JP1: Jumper_NO_Small, Jumper:SolderJumper-2_P1.3mm_Open_RoundedPad1.0x1.5mm, symbol Device:Jumper_NC_Small
- added Q10: FQP27P06, Package_TO_SOT_THT:TO-220-3_Horizontal_TabUp, symbol Transistor_FET:FQP27P06
- added Q9: BC807, Package_TO_SOT_SMD:SOT-23, symbol Transistor_BJT:BC807
- added R5, R6: 22k, Resistor_SMD:R_0805_2012Metric, symbol Arduino_Spot_Welderparts:R
- added R7: 33k, Resistor_SMD:R_0805_2012Metric, symbol Arduino_Spot_Welderparts:R
- added R8: 10k, Resistor_SMD:R_0805_2012Metric, symbol Arduino_Spot_Welderparts:R
- P1: value CONN_01X08 -> CONN_01X09; footprint Connector_JST:JST_XH_B8B-XH-A_1x08_P2.50mm_Vertical -> Connector_JST:JST_XH_B10B-XH-A_1x10_P2.50mm_Vertical; symbol Arduino_Spot_Welderparts:CONN_01X08 -> Connector:Conn_01x10_Male
Connections:
- net labels added: EnablePower, V_Batt
- wire segments 214 -> 218
Other:
- moved on the sheet: C12, C13, C14, D2, F1, H1, H2, H3, H4, H5, H6, H7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

Commit message: shunt replace
Parts:
- removed Q9: BC807, Package_TO_SOT_SMD:SOT-23, symbol Transistor_BJT:BC807
- removed R1: R_Shunt, SamacSys_Parts:WSK12161L000FEA, symbol Device:R_Shunt
- added IC1: INA213AIDCKR, SOT65P210X110-6N, symbol SamacSys_Parts:INA210AIDCKR
- added Q9: BC817, Package_TO_SOT_SMD:SOT-23, symbol Transistor_BJT:BC817
- added R1: 100µ, Resistor_SMD:R_Shunt_Vishay_WSR2_WSR3, symbol SamacSys_Parts:WSLP5931L1000FEA
- added R10: 30, Resistor_SMD:R_0805_2012Metric, symbol Arduino_Spot_Welderparts:R
- added R11, R12: 30k, Resistor_SMD:R_0805_2012Metric, symbol Arduino_Spot_Welderparts:R
- added R2: 10k, Resistor_SMD:R_0805_2012Metric, symbol Arduino_Spot_Welderparts:R
- added R9: 100, Resistor_SMD:R_0805_2012Metric, symbol Arduino_Spot_Welderparts:R
- added U2: LM4040DBZ-2.0, Package_TO_SOT_SMD:SOT-23, symbol Reference_Voltage:LM4040DBZ-2.0
- P1: footprint Connector_JST:JST_XH_B10B-XH-A_1x10_P2.50mm_Vertical -> Connector_JST:JST_XH_B9B-XH-A_1x09_P2.50mm_Vertical; symbol Connector:Conn_01x10_Male -> Connector:Conn_01x09_Male
Connections:
- net labels added: R_Schunt_Stab
- net labels removed: R_Schunt_H, R_Schunt_L
- wire segments 218 -> 244
Other:
- note added: "convert gain down to 20\n"

Commit message: pcb update 1.9
Parts:
- removed R10: 30, Resistor_SMD:R_0805_2012Metric, symbol Arduino_Spot_Welderparts:R
- removed R9: 100, Resistor_SMD:R_0805_2012Metric, symbol Arduino_Spot_Welderparts:R
- removed U2: LM4040DBZ-2.0, Package_TO_SOT_SMD:SOT-23, symbol Reference_Voltage:LM4040DBZ-2.0
- added C11, C?: 100n, Capacitor_SMD:C_0805_2012Metric_Pad1.18x1.45mm_HandSolder, symbol Device:C
- added C?: 1µ, Capacitor_SMD:C_1206_3216Metric, symbol Device:C
- added C?: 10n, Capacitor_SMD:C_0805_2012Metric_Pad1.18x1.45mm_HandSolder, symbol Device:C
- added U2: REF3020, Package_TO_SOT_SMD:SOT-23, symbol Reference_Voltage:REF3020
- Q10: footprint Package_TO_SOT_THT:TO-220-3_Horizontal_TabUp -> Package_TO_SOT_THT:TO-220-3_Horizontal_TabDown
- R11, R12: value 30k -> 12
- R7: value 33k -> 15k
- R8: value 10k -> 2.5k
Connections:
- net +5V: now also C?.2, U2.1 (IN)
- net GND: now also C11.2, C?.1, C?.2, U2.3 (GND)
- net V_Batt: now also C?.1
- net at IC1.4 (IN+), R11.1: now also C?.2
- net at IC1.5 (IN-), R12.1: now also C?.1
- net at IC1.1 (REF): now also C11.1, U2.2 (OUT)
Other:
- note added: "6.5kHz\n20V MAX"
- note added: "6.5khz\n"
- note removed: "convert gain down to 20\n"
- moved on the sheet: IC1, R11, R12

Commit message: PCB v2 , Power PCB routed
Parts:
- removed H1, H4: MountingHole_Pad, MountingHole:MountingHole_5.3mm_M5_Pad_Via, symbol Mechanical:MountingHole_Pad
- removed H2, H7: MountingHole_Pad, MountingHole:MountingHole_3.2mm_M3_Pad_Via, symbol Mechanical:MountingHole_Pad
- removed JP1: Jumper_NO_Small, Jumper:SolderJumper-2_P1.3mm_Open_RoundedPad1.0x1.5mm, symbol Device:Jumper_NC_Small
- removed R1: 100µ, Resistor_SMD:R_Shunt_Vishay_WSR2_WSR3, symbol SamacSys_Parts:WSLP5931L1000FEA
- removed R4: 10k, Resistor_SMD:R_0805_2012Metric, symbol Arduino_Spot_Welderparts:R
- removed U2: REF3020, Package_TO_SOT_SMD:SOT-23, symbol Reference_Voltage:REF3020
- added F2, F3, F4: 50A, my_parts:IMAXX_H1810-2x4, symbol Device:Fuse
- added J2: probe+, MountingHole:MountingHole_5.3mm_M5_Pad_Via, symbol Connector_Generic:Conn_01x01
- added J3, J6: Conn_01x02_Male, my_parts:AMASS_XT60-M_1x02_P7.20mm_Vertical, symbol Connector:Conn_01x02_Male
- added R1: 15k, Resistor_SMD:R_0805_2012Metric, symbol Arduino_Spot_Welderparts:R
- added R9: 2.5k, Resistor_SMD:R_0805_2012Metric, symbol Arduino_Spot_Welderparts:R
- C11: value 100n -> 10n
- C17: renamed from C?; footprint Capacitor_SMD:C_1206_3216Metric -> Capacitor_SMD:C_0805_2012Metric_Pad1.18x1.45mm_HandSolder
- D2: footprint Diode_SMD:D_SMA -> Diode_SMD:D_SMA_Handsoldering
- F1: value 300A -> 50A; footprint my_parts:ANL_Fuse -> my_parts:IMAXX_H1810-2x4
- gave numbers to parts that had none: 2
Connections:
- net +BATT: now also R11.2, F2.2, F3.2, F4.2, J3.2 (Pin_2), J6.2 (Pin_2)
- net Dallas: now also P1.7 (Pin_7); no longer P1.4 (Pin_4)
- net EnablePower: now also P1.4 (Pin_4); no longer P1.7 (Pin_7)
- net GND: now also D1.2 (A), H5.1, H6.1, IC1.1 (REF), Q1.3 (S), Q2.3 (S), Q3.3 (S), Q4.3 (S), Q5.3 (S), Q6.3 (S), Q7.3 (S), Q8.3 (S), J3.1 (Pin_1), J6.1 (Pin_1), R9.2; no longer R12.2
- net Gate_logic: now also P1.5 (Pin_5); no longer P1.3 (Pin_3)
- net Probe-: now also R1.1; no longer P1.5 (Pin_5)
- net R_Schunt_Stab: now also P1.2 (Pin_2); no longer P1.9 (Pin_9)
- net VCC: now also P1.9 (Pin_9); no longer IC3.1 (ENA), IC3.8 (ENB), P1.2 (Pin_2)
- net VCCQ: now also R12.2, F2.1, F3.1, F4.1, J2.1 (Pin_1)
- net V_Batt: now also P1.3 (Pin_3); no longer P1.6 (Pin_6)
- net at IC2.1 (ENA): no longer IC2.8 (ENB)
- net ProbeADC: now reaches C11.1
- net ProbeADC: now also P1.8 (Pin_8), R1.2, R9.1; no longer IC1.1 (REF)
- net +5V renamed +3V3
- net +3V3: now also P1.6 (Pin_6); no longer P1.8 (Pin_8)
- removed net FET_GND: D1.2 (A), H5.1, H6.1, Q1.3 (S), Q2.3 (S), Q3.3 (S), Q4.3 (S), Q5.3 (S), Q6.3 (S), Q7.3 (S), Q8.3 (S), R11.2
- no-connect marks 0 -> 4
Other:
- moved on the sheet: C16, C17, F1, IC1, P1, R11, R12

Commit message: clean up
Parts:
- added J5: TestCurr, Connector_PinHeader_2.54mm:PinHeader_1x02_P2.54mm_Vertical, symbol Connector:Conn_01x02_Male
Connections:
- net at C17.2, IC1.4 (IN+), R11.1: now also J5.1 (Pin_1)
- net at C17.1, IC1.5 (IN-), R12.1: now also J5.2 (Pin_2)
Changed lines of the file:
@@
 Connection ~ 6050 1050
 Wire Wire Line
-	5300 1350 5750 1350
+	5300 1350 5550 1350
 $Comp
 L power:+BATT #PWR0104
@@
 	6900 4600 6900 5650
 $Comp
-L power:GND #PWR?
+L power:GND #PWR0101
 U 1 1 61A575A8
 P 7700 3200
-F 0 "#PWR?" H 7700 2950 50  0001 C CNN
+F 0 "#PWR0101" H 7700 2950 50  0001 C CNN
 F 1 "GND" H 7705 3027 50  0000 C CNN
 F 2 "" H 7700 3200 50  0001 C CNN
@@
 	7700 3000 8100 3000
 Connection ~ 8100 3000
+$Comp
+L Connector:Conn_01x02_Male J5
+U 1 1 61B1CC3E
+P 10500 3150
+F 0 "J5" H 10472 3032 50  0000 R CNN
+F 1 "TestCurr" H 10472 3123 50  0000 R CNN
+F 2 "Connector_PinHeader_2.54mm:PinHeader_1x02_P2.54mm_Vertical" H 10500 3150 50  0001 C CNN
+F 3 "~" H 10500 3150 50  0001 C CNN
+	1    10500 3150
+	-1   0    0    1
+$EndComp
+Wire Wire Line
+	10300 3050 10300 3000
+Wire Wire Line
+	10300 3000 9700 3000
+Connection ~ 9700 3000
+Wire Wire Line
+	10300 3150 10300 3300
+Wire Wire Line
+	10300 3300 9700 3300
+Connection ~ 9700 3300
+$Comp
+L power:PWR_FLAG #FLG0101
+U 1 1 61B5E2BC
+P 5550 1250
+F 0 "#FLG0101" H 5550 1325 50  0001 C CNN
+F 1 "PWR_FLAG" H 5550 1423 50  0000 C CNN
+F 2 "" H 5550 1250 50  0001 C CNN
+F 3 "~" H 5550 1250 50  0001 C CNN
+	1    5550 1250
+	1    0    0    -1
+$EndComp
+Wire Wire Line
+	5550 1250 5550 1350
+Connection ~ 5550 1350
+Wire Wire Line
+	5550 1350 5750 1350
 $EndSCHEMATC

Commit message: V2 tweaks and tricks
Voltmeasure enable
Parts:
- removed J5: TestCurr, Connector_PinHeader_2.54mm:PinHeader_1x02_P2.54mm_Vertical, symbol Connector:Conn_01x02_Male
- added C18: 470p, Capacitor_SMD:C_0805_2012Metric_Pad1.18x1.45mm_HandSolder, symbol Device:C
- added Q11: BC817, Package_TO_SOT_SMD:SOT-23, symbol Transistor_BJT:BC817
- added Q12: BC807, Package_TO_SOT_SMD:SOT-23, symbol Transistor_BJT:BC807
- added R10: 470, Resistor_SMD:R_0805_2012Metric, symbol Arduino_Spot_Welderparts:R
- added R13, R14: 47k, Resistor_SMD:R_0805_2012Metric, symbol Arduino_Spot_Welderparts:R
- added R4: 10k, Resistor_SMD:R_0805_2012Metric, symbol Arduino_Spot_Welderparts:R
- C17: value 1µ -> 470p
- R11: value 12 -> 47k
- R12: value 12 -> 10k
Connections:
- net +BATT: now also IC1.4 (IN+); no longer R11.2
- net EnablePower: now also R4.1
- net GND: now also C17.2, C18.2, Q11.2 (E), R10.2
- net R_Schunt_Stab: now also C17.1, R13.2; no longer IC1.6 (OUT)
- net VCC: now also IC2.1 (ENA), IC2.8 (ENB), IC3.1 (ENA), IC3.8 (ENB)
- net VCCQ: now also IC1.5 (IN-), R11.1, Q12.3 (C); no longer R12.2
- net V_Batt: now also R14.2; no longer R7.2, R8.1
- net at D2.2 (A), Q10.2 (D): no longer R7.1
- net at Q9.1 (B), R2.1, R5.2: now also C18.1
- new net: Q12.2 (E), R7.1
- new net: R14.1, R7.2, R8.1
- new net: IC1.6 (OUT), R13.1
- new net: Q11.1 (B), R10.1, R4.2
- new net: Q11.3 (C), R12.2
- new net: Q12.1 (B), R11.2, R12.1
- no-connect marks 4 -> 0
Other:
- moved on the sheet: C14, C15, D2, R7, R8
