File: PCB/Spotwelderix/Spotwelderix.sch (KiCad schematic (older format))
At the start: 64 parts, among them IC1 INA213AIDCKR, IC2 IXDD604SIA, IC3 IXDD604SIA, J1 OnOffTast, J2 probe+, J3 Conn_01x02_Male, J4 probe-, J6 Conn_01x02_Male, P1 CONN_01X09, Q1 IRFB7430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

Commit message: connector sideflip
Parts:
- added R15: 47k, Resistor_SMD:R_0805_2012Metric, symbol Arduino_Spot_Welderparts:R
- J1: footprint Connector_JST:JST_XH_B2B-XH-A_1x02_P2.50mm_Vertical -> Connector_JST:JST_XH_S2B-XH-A_1x02_P2.50mm_Horizontal
Connections:
- net ProbeADC: now also R15.2; no longer R1.2, R9.1
- new net: R1.2, R15.1, R9.1
Other:
- moved on the sheet: C11
Changed lines of the file:
@@
 F 0 "J1" H 5808 1981 50  0000 C CNN
 F 1 "OnOffTast" H 5808 1890 50  0000 C CNN
-F 2 "Connector_JST:JST_XH_B2B-XH-A_1x02_P2.50mm_Vertical" H 5700 1800 50  0001 C CNN
+F 2 "Connector_JST:JST_XH_S2B-XH-A_1x02_P2.50mm_Horizontal" H 5700 1800 50  0001 C CNN
 F 3 "~" H 5700 1800 50  0001 C CNN
 	1    5700 1800
@@
 	8100 3000 8100 3100
 Connection ~ 8100 3100
-Text GLabel 4500 1350 2    50   Input ~ 0
+Text GLabel 4650 1350 2    50   Input ~ 0
 ProbeADC
 $Comp
@@
 	1    0    0    -1
 $EndComp
-Wire Wire Line
-	3900 1300 3900 1350
 $Comp
 L power:GND #PWR010
@@
 Wire Wire Line
 	3900 1950 3900 1800
-Wire Wire Line
-	3900 1350 4200 1350
-Connection ~ 3900 1350
-Wire Wire Line
-	3900 1350 3900 1450
-Text Notes 4150 1250 0    50   ~ 0
+Text Notes 4300 1200 0    50   ~ 0
 6.5kHz\n20V MAX
 $Comp
 L Device:C C11
 U 1 1 616258CF
-P 4200 1650
-F 0 "C11" H 4400 1650 50  0000 L CNN
-F 1 "10n" H 4300 1550 50  0000 L CNN
-F 2 "Capacitor_SMD:C_0805_2012Metric_Pad1.18x1.45mm_HandSolder" H 4238 1500 50  0001 C CNN
-F 3 "https://www.mouser.de/ProductDetail/Samsung-Electro-Mechanics/CL31A106KBHNNNE/?qs=sGAEpiMZZMuMW9TJLBQkXpvci%252BYHLlg21rnqFxf28Ww%3D" H 4200 1650 50  0001 C CNN
-	1    4200 1650
-	1    0    0    -1
-$EndComp
-Wire Wire Line
-	4200 1800 3900 1800
+P 4450 1650
+F 0 "C11" H 4650 1650 50  0000 L CNN
+F 1 "10n" H 4550 1550 50  0000 L CNN
+F 2 "Capacitor_SMD:C_0805_2012Metric_Pad1.18x1.45mm_HandSolder" H 4488 1500 50  0001 C CNN
+F 3 "https://www.mouser.de/ProductDetail/Samsung-Electro-Mechanics/CL31A106KBHNNNE/?qs=sGAEpiMZZMuMW9TJLBQkXpvci%252BYHLlg21rnqFxf28Ww%3D" H 4450 1650 50  0001 C CNN
+	1    4450 1650
+	1    0    0    -1
+$EndComp
 Connection ~ 3900 1800
 Wire Wire Line
 	3900 1800 3900 1750
-Wire Wire Line
-	4200 1500 4200 1350
-Connection ~ 4200 1350
-Wire Wire Line
-	4200 1350 4500 1350
 Text GLabel 3750 950  0    50   Input ~ 0
 Probe-
@@
 	6700 2350 6650 2350
 Connection ~ 6650 2350
+$Comp
+L Arduino_Spot_Welderparts:R R15
+U 1 1 6184EC9C
+P 4150 1350
+F 0 "R15" H 4220 1396 50  0000 L CNN
+F 1 "47k" H 4220 1305 50  0000 L CNN
+F 2 "Resistor_SMD:R_0805_2012Metric" H 4220 1259 50  0001 L CNN
+F 3 "" H 4150 1350 50  0000 C CNN
+	1    4150 1350
+	0    -1   -1   0
+$EndComp
+Wire Wire Line
+	3900 1300 3900 1350
+Wire Wire Line
+	4000 1350 3900 1350
+Connection ~ 3900 1350
+Wire Wire Line
+	3900 1350 3900 1450
+Wire Wire Line
+	4300 1350 4450 1350
+Wire Wire Line
+	4450 1500 4450 1350
+Connection ~ 4450 1350
+Wire Wire Line
+	4450 1350 4650 1350
+Wire Wire Line
+	3900 1800 4450 1800
 $EndSCHEMATC

Commit message: mount hole m4
Parts:
- H3, H5, H6: footprint MountingHole:MountingHole_5.3mm_M5_Pad_Via -> MountingHole:MountingHole_4.3mm_M4_Pad_Via
Changed lines of the file:
@@
 F 0 "H3" H 4550 6549 50  0000 L CNN
 F 1 "MountingHole_Pad" H 4550 6458 50  0000 L CNN
-F 2 "MountingHole:MountingHole_5.3mm_M5_Pad_Via" H 4450 6500 50  0001 C CNN
+F 2 "MountingHole:MountingHole_4.3mm_M4_Pad_Via" H 4450 6500 50  0001 C CNN
 F 3 "~" H 4450 6500 50  0001 C CNN
 	1    4450 6500
@@
 F 0 "H5" H 4100 7149 50  0000 L CNN
 F 1 "MountingHole_Pad" H 4100 7058 50  0000 L CNN
-F 2 "MountingHole:MountingHole_5.3mm_M5_Pad_Via" H 4000 7100 50  0001 C CNN
+F 2 "MountingHole:MountingHole_4.3mm_M4_Pad_Via" H 4000 7100 50  0001 C CNN
 F 3 "~" H 4000 7100 50  0001 C CNN
 	1    4000 7100
@@
 F 0 "H6" H 4600 7149 50  0000 L CNN
 F 1 "MountingHole_Pad" H 4600 7058 50  0000 L CNN
-F 2 "MountingHole:MountingHole_5.3mm_M5_Pad_Via" H 4500 7100 50  0001 C CNN
+F 2 "MountingHole:MountingHole_4.3mm_M4_Pad_Via" H 4500 7100 50  0001 C CNN
 F 3 "~" H 4500 7100 50  0001 C CNN
 	1    4500 7100

Commit message: SW auto calibrate batt volt
Parts:
- R10: value 470 -> 47k
Connections:
- net VCCQ: no longer R11.1
- net at Q12.2 (E), R7.1: now also R11.1
Other:
- moved on the sheet: R11
Changed lines of the file:
@@
 P 3900 1150
 F 0 "R1" H 3970 1196 50  0000 L CNN
-F 1 "15k" H 3970 1105 50  0000 L CNN
+F 1 "15k" H 4000 1250 50  0000 L CNN
 F 2 "Resistor_SMD:R_0805_2012Metric" H 3970 1059 50  0001 L CNN
 F 3 "" H 3900 1150 50  0000 C CNN
@@
 P 9350 1950
 F 0 "R10" H 9420 1996 50  0000 L CNN
-F 1 "470" H 9420 1905 50  0000 L CNN
+F 1 "47k" H 9420 1905 50  0000 L CNN
 F 2 "Resistor_SMD:R_0805_2012Metric" H 9420 1859 50  0001 L CNN
 F 3 "" H 9350 1950 50  0000 C CNN
@@
 L Arduino_Spot_Welderparts:R R11
 U 1 1 6152C3FA
-P 9450 900
-F 0 "R11" H 9520 946 50  0000 L CNN
-F 1 "47k" H 9520 855 50  0000 L CNN
-F 2 "Resistor_SMD:R_0805_2012Metric" H 9520 809 50  0001 L CNN
-F 3 "" H 9450 900 50  0000 C CNN
-	1    9450 900
-	1    0    0    -1
+P 10100 1100
+F 0 "R11" H 9900 1200 50  0000 L CNN
+F 1 "47k" H 9900 1100 50  0000 L CNN
+F 2 "Resistor_SMD:R_0805_2012Metric" H 10170 1009 50  0001 L CNN
+F 3 "" H 10100 1100 50  0000 C CNN
+	1    10100 1100
+	0    1    1    0
 $EndComp
 $Comp
@@
 	10100 750  10300 750
 Wire Wire Line
-	10300 750  10300 1150
-Wire Wire Line
-	9900 1050 9900 1100
+	10300 750  10300 1100
 Wire Wire Line
 	9900 1450 9900 1550
 Wire Wire Line
-	9450 750  9700 750
-Wire Wire Line
-	9900 1100 9450 1100
-Wire Wire Line
-	9450 1100 9450 1050
-Connection ~ 9900 1100
-Wire Wire Line
-	9900 1100 9900 1150
-Wire Wire Line
-	9450 750  7300 750
-Wire Wire Line
 	7300 750  7300 900
 Wire Wire Line
 	7300 900  6350 900
-Connection ~ 9450 750
 Connection ~ 6350 900
 Wire Wire Line
@@
 Wire Wire Line
 	3900 1800 4450 1800
+Wire Wire Line
+	9900 1050 9900 1100
+Wire Wire Line
+	7300 750  9700 750
+Wire Wire Line
+	9950 1100 9900 1100
+Connection ~ 9900 1100
+Wire Wire Line
+	9900 1100 9900 1150
+Wire Wire Line
+	10250 1100 10300 1100
+Connection ~ 10300 1100
+Wire Wire Line
+	10300 1100 10300 1150
 $EndSCHEMATC

Commit message: v4
Parts:
- removed F2, F3: 50A, my_parts:IMAXX_H1810-2x4, symbol Device:Fuse
- removed IC1: INA213AIDCKR, SOT65P210X110-6N, symbol SamacSys_Parts:INA210AIDCKR
- removed IC2, IC3: IXDD604SIA, SamacSys_Parts:SOIC127P600X175-8N, symbol SamacSys_Parts:IXDD604SIA
- removed Q11: BC817, Package_TO_SOT_SMD:SOT-23, symbol Transistor_BJT:BC817
- removed Q12: BC807, Package_TO_SOT_SMD:SOT-23, symbol Transistor_BJT:BC807
- removed R12: 10k, Resistor_SMD:R_0805_2012Metric, symbol Arduino_Spot_Welderparts:R
- removed R14: 47k, Resistor_SMD:R_0805_2012Metric, symbol Arduino_Spot_Welderparts:R
- added C19: 10µ, Capacitor_SMD:C_1206_3216Metric, symbol Device:C
- added IC1, IC2: IXDD604SIA, SOIC127P600X175-8N, symbol mouser:IXDD604SIA
- added Q11, Q12: DMG3402_SOT23_n_Fet_3A, Package_TO_SOT_SMD:SOT-23_Handsoldering, symbol my_parts:DMG3402_SOT23_n_Fet_3A
- added U2, U3: AD8209, Package_SO:MSOP-8_3x3mm_P0.65mm, symbol Amplifier_Current:AD8209
- C15: value 10n -> 470p
- C16: value 100n -> 10µ; footprint Capacitor_SMD:C_0805_2012Metric_Pad1.18x1.45mm_HandSolder -> Capacitor_SMD:C_1206_3216Metric
- F1, F4: footprint my_parts:IMAXX_H1810-2x4 -> my_parts:Blade_Fuse_maxi_handsolder_1.5drill
- J3, J6: value Conn_01x02_Male -> XT90
- R10: value 47k -> 100
- R11, R13: value 47k -> 55k
- R4: value 10k -> 100
- R7: value 15k -> 133k
- R8: value 2.5k -> 100
Connections:
- net +BATT: now also U2.8 (+IN)
- net Dallas: now also R8.1; no longer U1.2 (DQ)
- net EnablePower: now also Q11.1; no longer R4.1
- net GND: now also C16.2, R11.2, C19.2, IC1.3 (GND), IC2.3 (GND), Q11.2, Q12.2, U2.2 (GND), U3.2 (GND); no longer C11.2, C16.1, R10.2, R8.2, R9.2
- net Gate: now also IC1.5 (OUTB), IC1.7 (OUTA), IC2.5 (OUTB), IC2.7 (OUTA)
- net Gate_logic: now also IC1.2 (INA), IC1.4 (INB), IC2.2 (INA), IC2.4 (INB), Q12.1
- net Probe-: now also U3.1 (-IN)
- net R_Schunt_Stab: now also R10.2; no longer C17.1, R13.2
- net VCC: now also IC1.1 (ENA), IC1.6 (VCC), IC1.8 (ENB), IC2.1 (ENA), IC2.6 (VCC), IC2.8 (ENB)
- net VCCQ: now also U2.1 (-IN), U3.8 (+IN)
- net at R11.1: now also C15.1, R7.2, U3.3 (A1), U3.4 (A2); no longer R7.1
- net at R13.1: now also C17.1, U2.3 (A1), U2.4 (A2)
- net at R10.1: now also U2.5 (OUT); no longer R4.2
- net +3V3 renamed +5V
- net +5V: now also C16.1, C19.1, U2.7 (+Vs), U3.7 (+Vs); no longer C16.2
- net V_Batt renamed Probe_diff
- net Probe_diff: now also R4.1; no longer C15.1
- new net: R8.2, U1.2 (DQ)
- new net: Q12.3, R13.2
- new net: C11.2, Q11.3, R9.2
- new net: R4.2, R7.1, U3.5 (OUT)
Other:
- note added: "gain 5, Rext = 55k\nwhile gate active only"
- note added: "gain 50, Rext = 133k\n"
- note removed: "6.5khz\n"
- moved on the sheet: C1, C10, C11, C12, C13, C14, C17, C18, C2, C3, C4, C5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

Commit message: auto weld, non functional
Parts:
- R11: value 55k -> 2k5
- R7: value 133k -> 15k
Connections:
- net +5V: no longer U3.7 (+Vs)
- net GND: no longer U3.2 (GND)
- net VCCQ: now also R7.1; no longer U3.8 (+IN)
- net at C15.1, R11.1, R7.2: now also R4.2; no longer U3.3 (A1), U3.4 (A2)
- now unconnected: U3.5 (OUT)
Other:
- note added: "gain = 1\nRext = 7.1"
- moved on the sheet: C15, J4, R11, R4, U3
Changed lines of the file:
@@
 L Connector_Generic:Conn_01x01 J4
 U 1 1 6027240D
-P 6300 3550
-F 0 "J4" H 6380 3592 50  0000 L CNN
-F 1 "probe-" H 6380 3501 50  0000 L CNN
-F 2 "MountingHole:MountingHole_5.3mm_M5_Pad_Via" H 6300 3550 50  0001 C CNN
-F 3 "~" H 6300 3550 50  0001 C CNN
-	1    6300 3550
+P 5750 3550
+F 0 "J4" H 5830 3592 50  0000 L CNN
+F 1 "probe-" H 5830 3501 50  0000 L CNN
+F 2 "MountingHole:MountingHole_5.3mm_M5_Pad_Via" H 5750 3550 50  0001 C CNN
+F 3 "~" H 5750 3550 50  0001 C CNN
+	1    5750 3550
 	1    0    0    -1
 $EndComp
@@
 	1    0    0    -1
 $EndComp
-Wire Wire Line
-	6100 3550 6050 3550
 Connection ~ 4250 3550
 Wire Wire Line
@@
 L Amplifier_Current:AD8209 U3
 U 1 1 61E0AEFA
-P 5850 4350
-F 0 "U3" H 5950 3850 50  0000 L CNN
-F 1 "AD8209" H 6000 3950 50  0000 L CNN
-F 2 "Package_SO:MSOP-8_3x3mm_P0.65mm" H 5900 4000 50  0001 L CNN
-F 3 "https://www.analog.com/media/en/technical-documentation/data-sheets/AD8209.pdf" H 6500 3650 50  0001 C CNN
-	1    5850 4350
+P 5200 4350
+F 0 "U3" H 5300 3850 50  0000 L CNN
+F 1 "AD8209" H 5350 3950 50  0000 L CNN
+F 2 "Package_SO:MSOP-8_3x3mm_P0.65mm" H 5250 4000 50  0001 L CNN
+F 3 "https://www.analog.com/media/en/technical-documentation/data-sheets/AD8209.pdf" H 5850 3650 50  0001 C CNN
+	1    5200 4350
 	1    0    0    -1
 $EndComp
@@
 L power:VCCQ #PWR0114
 U 1 1 61E1E268
-P 5650 3800
-F 0 "#PWR0114" H 5650 3650 50  0001 C CNN
-F 1 "VCCQ" H 5665 3973 50  0000 C CNN
-F 2 "" H 5650 3800 50  0001 C CNN
-F 3 "" H 5650 3800 50  0001 C CNN
-	1    5650 3800
-	1    0    0    -1
-$EndComp
-Wire Wire Line
-	5650 3950 5650 3800
-Wire Wire Line
-	6050 3950 6050 3550
+P 6800 4300
+F 0 "#PWR0114" H 6800 4150 50  0001 C CNN
+F 1 "VCCQ" H 6815 4473 50  0000 C CNN
+F 2 "" H 6800 4300 50  0001 C CNN
+F 3 "" H 6800 4300 50  0001 C CNN
+	1    6800 4300
+	1    0    0    -1
+$EndComp
+Wire Wire Line
+	6800 4450 6800 4300
 $Comp
 L power:GND #PWR0118
@@
 Wire Wire Line
 	7000 1050 8900 1050
-Text GLabel 6500 3900 2    50   Input ~ 0
+Text GLabel 5200 5400 0    50   Input ~ 0
 Probe_diff
 Text GLabel 2100 6900 0    50   Input ~ 0
@@
 L Arduino_Spot_Welderparts:R R4
 U 1 1 6202236D
-P 6350 4100
-F 0 "R4" H 6420 4146 50  0000 L CNN
-F 1 "100" H 6420 4055 50  0000 L CNN
-F 2 "Resistor_SMD:R_0805_2012Metric" H 6420 4009 50  0001 L CNN
-F 3 "" H 6350 4100 50  0000 C CNN
-	1    6350 4100
-	1    0    0    -1
-$EndComp
-Wire Wire Line
-	6250 4350 6350 4350
-Wire Wire Line
-	6350 4350 6350 4250
-Wire Wire Line
-	6350 3950 6350 3900
-Wire Wire Line
-	6350 3900 6500 3900
+P 5500 5400
+F 0 "R4" H 5570 5446 50  0000 L CNN
+F 1 "100" H 5570 5355 50  0000 L CNN
+F 2 "Resistor_SMD:R_0805_2012Metric" H 5570 5309 50  0001 L CNN
+F 3 "" H 5500 5400 50  0000 C CNN
+	1    5500 5400
+	0    -1   -1   0
+$EndComp
+Wire Wire Line
+	5350 5400 5200 5400
 $Comp
 L power:GND #PWR0123
 U 1 1 62054793
-P 5850 5150
-F 0 "#PWR0123" H 5850 4900 50  0001 C CNN
-F 1 "GND" H 5855 4977 50  0000 C CNN
-F 2 "" H 5850 5150 50  0001 C CNN
-F 3 "" H 5850 5150 50  0001 C CNN
-	1    5850 5150
-	1    0    0    -1
-$EndComp
-Wire Wire Line
-	5850 5150 5850 5050
-Wire Wire Line
-	5200 5050 5850 5050
-Connection ~ 5850 5050
-Wire Wire Line
-	5850 5050 5850 4750
-Connection ~ 6050 3550
-Wire Wire Line
-	4250 3550 6050 3550
+P 6050 5900
+F 0 "#PWR0123" H 6050 5650 50  0001 C CNN
+F 1 "GND" H 6055 5727 50  0000 C CNN
+F 2 "" H 6050 5900 50  0001 C CNN
+F 3 "" H 6050 5900 50  0001 C CNN
+	1    6050 5900
+	1    0    0    -1
+$EndComp
 $Comp
 L Device:C C15
 U 1 1 62088B6C
-P 5200 4750
-F 0 "C15" H 5300 4900 50  0000 L CNN
-F 1 "470p" H 5200 4600 50  0000 L CNN
-F 2 "Capacitor_SMD:C_0805_2012Metric_Pad1.18x1.45mm_HandSolder" H 5238 4600 50  0001 C CNN
-F 3 "https://www.mouser.de/ProductDetail/Samsung-Electro-Mechanics/CL31A106KBHNNNE/?qs=sGAEpiMZZMuMW9TJLBQkXpvci%252BYHLlg21rnqFxf28Ww%3D" H 5200 4750 50  0001 C CNN
-	1    5200 4750
-	1    0    0    -1
-$EndComp
-Wire Wire Line
-	5450 4450 5200 4450
-Wire Wire Line
-	5200 4450 5200 4350
-Wire Wire Line
-	5200 4350 5450 4350
-Wire Wire Line
-	5200 4450 5200 4600
-Connection ~ 5200 4450
-Wire Wire Line
-	5200 4900 5200 5050
-$Comp
-L power:+5V #PWR0124
-U 1 1 6209AE8B
-P 5600 4900
-F 0 "#PWR0124" H 5600 4750 50  0001 C CNN
-F 1 "+5V" H 5615 5073 50  0000 C CNN
-F 2 "" H 5600 4900 50  0001 C CNN
-F 3 "" H 5600 4900 50  0001 C CNN
-	1    5600 4900
-	1    0    0    -1
-$EndComp
-Wire Wire Line
-	5450 4950 5600 4950
-Wire Wire Line
-	5600 4950 5600 4900
-Wire Wire Line
-	5450 4550 5450 4950
+P 6050 5650
+F 0 "C15" H 6150 5800 50  0000 L CNN
+F 1 "470p" H 6050 5500 50  0000 L CNN
+F 2 "Capacitor_SMD:C_0805_2012Metric_Pad1.18x1.45mm_HandSolder" H 6088 5500 50  0001 C CNN
+F 3 "https://www.mouser.de/ProductDetail/Samsung-Electro-Mechanics/CL31A106KBHNNNE/?qs=sGAEpiMZZMuMW9TJLBQkXpvci%252BYHLlg21rnqFxf28Ww%3D" H 6050 5650 50  0001 C CNN
+	1    6050 5650
+	1    0    0    -1
+$EndComp
 Text Notes 6400 4750 0    50   ~ 0
 gain 50, Rext = 133k\n
@@
 P 6350 4900
 F 0 "R7" H 6420 4946 50  0000 L CNN
-F 1 "133k" H 6420 4855 50  0000 L CNN
+F 1 "15k" H 6420 4855 50  0000 L CNN
 F 2 "Resistor_SMD:R_0805_2012Metric" H 6420 4809 50  0001 L CNN
 F 3 "" H 6350 4900 50  0000 C CNN
@@
 	6350 5050 6350 5400
 Wire Wire Line
-	6350 5400 4950 5400
-Wire Wire Line
-	4950 5400 4950 4350
-Wire Wire Line
-	4950 4350 5200 4350
-Connection ~ 5200 4350
-Wire Wire Line
-	6350 4750 6350 4350
-Connection ~ 6350 4350
+	6350 5400 6050 5400
+Wire Wire Line
+	6350 4750 6350 4450
 $Comp
 L my_parts:DMG3402_SOT23_n_Fet_3A Q12
@@
 L Arduino_Spot_Welderparts:R R11
 U 1 1 619FF475
-P 4950 5650
-F 0 "R11" H 5020 5696 50  0000 L CNN
-F 1 "55k" H 5020 5605 50  0000 L CNN
-F 2 "Resistor_SMD:R_0805_2012Metric" H 5020 5559 50  0001 L CNN
-F 3 "" H 4950 5650 50  0000 C CNN
-	1    4950 5650
+P 6350 5650
+F 0 "R11" H 6420 5696 50  0000 L CNN
+F 1 "2k5" H 6420 5605 50  0000 L CNN
+F 2 "Resistor_SMD:R_0805_2012Metric" H 6420 5559 50  0001 L CNN
+F 3 "" H 6350 5650 50  0000 C CNN
+	1    6350 5650
 	1    0    0    -1
 $EndComp
@@
 L power:GND #PWR08
 U 1 1 61A13350
-P 4950 5900
-F 0 "#PWR08" H 4950 5650 50  0001 C CNN
-F 1 "GND" H 4955 5727 50  0000 C CNN
-F 2 "" H 4950 5900 50  0001 C CNN
-F 3 "" H 4950 5900 50  0001 C CNN
-	1    4950 5900
-	1    0    0    -1
-$EndComp
-Wire Wire Line
-	4950 5500 4950 5400
-Connection ~ 4950 5400
-Wire Wire Line
-	4950 5900 4950 5800
+P 6350 5900
+F 0 "#PWR08" H 6350 5650 50  0001 C CNN
+F 1 "GND" H 6355 5727 50  0000 C CNN
+F 2 "" H 6350 5900 50  0001 C CNN
+F 3 "" H 6350 5900 50  0001 C CNN
+	1    6350 5900
+	1    0    0    -1
+$EndComp
+Wire Wire Line
+	6350 5500 6350 5400
+Wire Wire Line
+	6350 5900 6350 5800
+Text Notes 5350 5850 0    50   ~ 0
+gain = 1\nRext = 7.1
+Wire Wire Line
+	6050 5900 6050 5800
+Wire Wire Line
+	6050 5500 6050 5400
+Wire Wire Line
+	6800 4450 6350 4450
+Wire Wire Line
+	5400 3950 5400 3550
+Wire Wire Line
+	4250 3550 5400 3550
+Wire Wire Line
+	5550 3550 5400 3550
+Connection ~ 5400 3550
+Connection ~ 6350 5400
+Wire Wire Line
+	5650 5400 6050 5400
+Connection ~ 6050 5400
 $EndSCHEMATC
